File: KiCAD/stm8-gamepad/nucleo-8s207k8.kicad_sch (KiCad schematic)
At the start: 20 parts, among them J10 video out, J7 batt., J8 batt., J9 audio out, SW10 UP, SW11 DOWN, SW12 RIGHT, SW13 B, SW14 A, SW8 power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

Commit message: Modification matérielle cristal de 16Mhz remplacé par 24Mhz. Amélioration du rapport largeur/hauteur de l'image maintenant proche de l'utnité
Parts:
- R5: value 150 -> 100
- Y2: value 16Mhz -> 24Mhz
Changed lines of the file:
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@@
     (in_bom yes) (on_board yes) (fields_autoplaced)
     (property "Reference" "Y2" (id 0) (at 114.3 118.11 0))
-    (property "Value" "16Mhz" (id 1) (at 114.3 120.65 0))
+    (property "Value" "24Mhz" (id 1) (at 114.3 120.65 0))
     (property "Footprint" "" (id 2) (at 114.3 125.73 0)
       (effects (font (size 1.27 1.27)) hide)
@@
     (in_bom yes) (on_board yes)
     (property "Reference" "R5" (id 0) (at 182.245 100.33 90))
-    (property "Value" "150" (id 1) (at 182.245 105.41 90))
+    (property "Value" "100" (id 1) (at 182.245 105.41 90))
     (property "Footprint" "" (id 2) (at 182.245 104.648 90)
       (effects (font (size 1.27 1.27)) hide)
